File: Flybot_FC/Flybot FC/src/Flybot_FC/32V-5V.3A_BuckConverter_SY8303.kicad_sch (KiCad schematic)
At the start: 23 parts, among them Q3 AO3401A, Q4 SI2301CDS-T1-GE3, U9 SY8303AIC

Commit message: Bill of materials
Parts:
- C75, C76: footprint Capacitor_SMD:C_0603_1608Metric -> Capacitor_SMD:C_0402_1005Metric
- D10: value B22AL2 -> D15V0S1U2LP1610-7; footprint (none) -> Diode_SMD:D_0603_1608Metric
- D8: value SS54F -> SDM4A40EP3-7B; footprint Diode_SMD:D_SMA -> Diode_SMD:D_0603_1608Metric
- D9: value BZT52C12 -> BZX884B30L-G3-08; footprint Diode_SMD:D_SOD-123 -> Diode_SMD:D_0402_1005Metric
- L4: footprint (none) -> Inductor_SMD:L_1210_3225Metric
- R34, R35, R36, R37, R39: footprint Resistor_SMD:R_0603_1608Metric -> Resistor_SMD:R_0402_1005Metric
- TP25, TP26: footprint (none) -> TestPoint:TestPoint_Pad_D1.0mm
- U9: value SY8303AIC -> SY21153AAIC; footprint Package_TO_SOT_SMD:TSOT-23-8_HandSoldering -> Package_TO_SOT_SMD:TSOT-23-8
