File: Flybot_FC/Flybot FC/src/Flybot_FC/5V-3.3V.3A_BuckConverter_SY8089.kicad_sch (KiCad schematic)
At the start: 14 parts, among them U10 SY8089AAAC

Commit message: Bill of materials
Parts:
- removed TP16: Sw, TestPoint:TestPoint_Pad_D1.0mm, symbol Connector:TestPoint
- R40: value 450k -> 453k
- TP27: footprint (none) -> TestPoint:TestPoint_Pad_D1.0mm
- U10: value SY8089AAAC -> RT5752AHGJ5
Changed lines of the file:
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@@
-	)
-	(junction
-		(at 149.86 74.93)
-		(diameter 0)
-		(color 0 0 0 0)
 	)
 	(junction
@@
 	(wire
 		(pts
-			(xy 149.86 74.93) (xy 152.4 74.93)
+			(xy 148.59 74.93) (xy 152.4 74.93)
 		)
 		(stroke
@@
 	(wire
 		(pts
-			(xy 148.59 74.93) (xy 149.86 74.93)
-		)
-		(stroke
-			(width 0)
-			(type default)
-		)
-	)
-	(wire
-		(pts
 			(xy 177.8 74.93) (xy 189.23 74.93)
-		)
-		(stroke
-			(width 0)
-			(type default)
-		)
-	)
-	(wire
-		(pts
-			(xy 149.86 69.85) (xy 149.86 74.93)
 		)
 		(stroke
@@
 		)
 		(property "Sim.Pins" ""
+			(at 78.74 81.28 0)
+			(effects
+				(font
+					(size 1.27 1.27)
+				)
+			)
+		)
+		(property "Field4" ""
 			(at 78.74 81.28 0)
 			(effects
@@
 			)
 		)
+		(property "Field4" ""
+			(at 96.52 81.28 0)
+			(effects
+				(font
+					(size 1.27 1.27)
+				)
+			)
+		)
 		(pin "2"
 		)
@@
 			)
 		)
+		(property "Field4" ""
+			(at 205.74 82.55 0)
+			(effects
+				(font
+					(size 1.27 1.27)
+				)
+			)
+		)
 		(pin "2"
 		)
@@
 		)
 		(property "Sim.Pins" ""
+			(at 189.23 82.55 0)
+			(effects
+				(font
+					(size 1.27 1.27)
+				)
+			)
+		)
+		(property "Field4" ""
 			(at 189.23 82.55 0)
 			(effects
@@
 			)
 		)
+		(property "Field4" ""
+			(at 205.74 69.85 0)
+			(effects
+				(font
+					(size 1.27 1.27)
+				)
+			)
+		)
 		(pin "1"
 		)
@@
 				(path "/376dca49-3f61-489b-8a1c-02451cc2f7ba/e434f21c-e709-4bca-915d-3aeda9c908e5"
 					(reference "TP16")
-					(unit 1)
-				)
-			)
-		)
-	)
-	(symbol
-		(lib_id "Connector:TestPoint")
-		(at 149.86 69.85 0)
-		(unit 1)
-		(exclude_from_sim no)
-		(in_bom yes)
-		(on_board yes)
-		(dnp no)
-		(property "Reference" "TP16"
-			(at 147.574 62.992 0)
-			(effects
-				(font
-					(size 1.27 1.27)
-				)
-				(justify left)
-			)
-		)
-		(property "Value" "Sw"
-			(at 148.336 64.77 0)
-			(effects
-				(font
-					(size 1.27 1.27)
-				)
-				(justify left)
-			)
-		)
-		(property "Footprint" "TestPoint:TestPoint_Pad_D1.0mm"
-			(at 154.94 69.85 0)
-			(effects
-				(font
-					(size 1.27 1.27)
-				)
-				(hide yes)
-			)
-		)
-		(property "Datasheet" "~"
-			(at 154.94 69.85 0)
-			(effects
-				(font
-					(size 1.27 1.27)
-				)
-				(hide yes)
-			)
-		)
-		(property "Description" "test point"
-			(at 149.86 69.85 0)
-			(effects
-				(font
-					(size 1.27 1.27)
-				)
-				(hide yes)
-			)
-		)
-		(property "Sim.Type" ""
-			(at 149.86 69.85 0)
-			(effects
-				(font
-					(size 1.27 1.27)
-				)
-			)
-		)
-		(property "Sim.Pins" ""
-			(at 149.86 69.85 0)
-			(effects
-				(font
-					(size 1.27 1.27)
-				)
-			)
-		)
-		(pin "1"
-		)
-		(instances
-			(project "Flybot_FC"
-				(path "/20662b15-1234-4fb8-8b52-cea64be60f62/1e2f80bf-4e41-4389-9b25-59776cd7a69e"
-					(reference "TP16")
-					(unit 1)
-				)
-			)
-			(project "SafiVolt_Main"
-				(path "/376dca49-3f61-489b-8a1c-02451cc2f7ba/e434f21c-e709-4bca-915d-3aeda9c908e5"
-					(reference "TP15")
 					(unit 1)
 				)
@@
 			)
 		)
+		(property "Field4" ""
+			(at 87.63 81.28 0)
+			(effects
+				(font
+					(size 1.27 1.27)
+				)
+			)
+		)
 		(pin "2"
 		)
@@
 			)
 		)
-		(property "Value" "SY8089AAAC"
+		(property "Value" "RT5752AHGJ5"
 			(at 138.43 70.866 0)
 			(effects
@@
 			)
 		)
-		(property "Datasheet" "https://www.lcsc.com/datasheet/lcsc_datasheet_2409291603_Silergy-Corp-SY8089AAAC_C78988.pdf"
+		(property "Datasheet" "https://www.richtek.com/assets/product_file/RT5752A=RT5752B/DS5752AB-02.pdf"
 			(at 137.668 68.326 0)
 			(effects
@@
 		)
 		(property "Sim.Pins" ""
+			(at 138.43 80.01 0)
+			(effects
+				(font
+					(size 1.27 1.27)
+				)
+			)
+		)
+		(property "Field4" ""
 			(at 138.43 80.01 0)
 			(effects
@@
 			)
 		)
-		(property "Footprint" ""
+		(property "Footprint" "TestPoint:TestPoint_Pad_D1.0mm"
 			(at 110.49 119.38 0)
 			(effects
@@
 				)
 				(hide yes)
+			)
+		)
+		(property "Field4" ""
+			(at 105.41 119.38 0)
+			(effects
+				(font
+					(size 1.27 1.27)
+				)
 			)
 		)
@@
 			)
 		)
+		(property "Field4" ""
+			(at 177.8 82.55 0)
+			(effects
+				(font
+					(size 1.27 1.27)
+				)
+			)
+		)
 		(pin "2"
 		)
@@
 			)
 		)
+		(property "Field4" ""
+			(at 166.37 93.98 0)
+			(effects
+				(font
+					(size 1.27 1.27)
+				)
+			)
+		)
 		(pin "1"
 		)
@@
 			)
 		)
-		(property "Value" "450k"
+		(property "Value" "453k"
 			(at 167.894 85.09 0)
 			(effects
@@
 		)
 		(property "Sim.Pins" ""
+			(at 166.37 83.82 0)
+			(effects
+				(font
+					(size 1.27 1.27)
+				)
+			)
+		)
+		(property "Field4" ""
 			(at 166.37 83.82 0)
 			(effects
@@
 			)
 		)
+		(property "Field4" ""
+			(at 156.21 74.93 0)
+			(effects
+				(font
+					(size 1.27 1.27)
+				)
+			)
+		)
 		(pin "2"
 		)
@@
 			(at 198.12 82.55 0)
 			(effects
+				(font
+					(size 1.27 1.27)
+				)
+			)
+		)
+		(property "Field4" ""
+			(at 198.12 82.55 0)
+			(effects
