File: Flybot_FC/Flybot FC/src/Flybot_FC/Flybot_FC.kicad_sch (KiCad schematic)
At the start: 4 parts

Commit message: Bill of materials
Parts:
- H1, H2, H3, H4: footprint (none) -> MountingHole:MountingHole_3mm
Changed lines of the file:
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@@
 			)
 		)
-		(property "Footprint" ""
+		(property "Footprint" "MountingHole:MountingHole_3mm"
 			(at 92.71 186.69 0)
 			(effects
@@
 				)
 				(hide yes)
+			)
+		)
+		(property "Field4" ""
+			(at 92.71 186.69 0)
+			(effects
+				(font
+					(size 1.27 1.27)
+				)
 			)
 		)
@@
 			)
 		)
-		(property "Footprint" ""
+		(property "Footprint" "MountingHole:MountingHole_3mm"
 			(at 92.71 177.8 0)
 			(effects
@@
 				)
 				(hide yes)
+			)
+		)
+		(property "Field4" ""
+			(at 92.71 177.8 0)
+			(effects
+				(font
+					(size 1.27 1.27)
+				)
 			)
 		)
@@
 			)
 		)
-		(property "Footprint" ""
+		(property "Footprint" "MountingHole:MountingHole_3mm"
 			(at 69.85 177.8 0)
 			(effects
@@
 				)
 				(hide yes)
+			)
+		)
+		(property "Field4" ""
+			(at 69.85 177.8 0)
+			(effects
+				(font
+					(size 1.27 1.27)
+				)
 			)
 		)
@@
 			)
 		)
-		(property "Footprint" ""
+		(property "Footprint" "MountingHole:MountingHole_3mm"
 			(at 69.85 186.69 0)
 			(effects
@@
 			)
 		)
+		(property "Field4" ""
+			(at 69.85 186.69 0)
+			(effects
+				(font
+					(size 1.27 1.27)
+				)
+			)
+		)
