File: Flybot_FC/Flybot FC/src/Flybot_FC/LSM6DSOX_IMU.kicad_sch (KiCad schematic)
At the start: 8 parts, among them U6 LSM6DSOX, U7 LSM6DSOX

Commit message: Bill of materials
Parts:
- removed U7: LSM6DSOX, Package_LGA:LGA-14_3x2.5mm_P0.5mm_LayoutBorder3x4y, symbol Sensor_Motion:LSM6DS3
- added U7: ICM-42688P-HXY, Package_LGA:LGA-14_3x2.5mm_P0.5mm_LayoutBorder3x4y, symbol Sensor_Motion:ICM-20602
- C65, C66, C67, C68, C69, C70: footprint (none) -> Capacitor_SMD:C_0402_1005Metric
Connections:
- net +3V3: now also U7.5 (VDDIO), U7.8 (VDD)
- net GND: now also U7.10 (RESV), U7.11 (RESV), U7.2 (RESV), U7.3 (RESV), U7.6 (GND), U7.7 (RESV)
- net IMU2.CS: now also U7.12 (AP_CS)
- net IMU2_INT: now also U7.4 (INT1)
- net MISO: now also U7.1 (AP_SDO)
- net MOSI: now also U7.14 (AP_SDI)
- net SCLK: now also U7.13 (AP_SCLK)
