File: Flybot_FC/Flybot FC/src/Flybot_FC/W25Q128JVE_FLASH.MEMORY.kicad_sch (KiCad schematic)
At the start: 6 parts, among them U11 W25Q128JVE

Commit message: Bill of materials
Parts:
- U11: value W25Q128JVE -> AT25SF128A-MHB-T; footprint Package_SON:WSON-8-1EP_8x6mm_P1.27mm_EP3.4x4.3mm -> Package_DFN_QFN:DFN-8-1EP_6x5mm_P1.27mm_EP4x4mm
Changed lines of the file:
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@@
+			)
+		)
+		(property "Field4" ""
+			(at 138.43 83.82 0)
+			(effects
+				(font
+					(size 1.27 1.27)
+				)
 			)
 		)
@@
 		)
 		(property "LCSC" ""
+			(at 110.49 113.03 0)
+			(effects
+				(font
+					(size 1.27 1.27)
+				)
+			)
+		)
+		(property "Field4" ""
 			(at 110.49 113.03 0)
 			(effects
@@
 			)
 		)
+		(property "Field4" ""
+			(at 110.49 110.49 0)
+			(effects
+				(font
+					(size 1.27 1.27)
+				)
+			)
+		)
 		(pin "1"
 		)
@@
 			)
 		)
+		(property "Field4" ""
+			(at 148.59 83.82 0)
+			(effects
+				(font
+					(size 1.27 1.27)
+				)
+			)
+		)
 		(pin "1"
 		)
@@
 			)
 		)
+		(property "Field4" ""
+			(at 111.76 88.9 0)
+			(effects
+				(font
+					(size 1.27 1.27)
+				)
+			)
+		)
 		(pin "2"
 		)
@@
 			)
 		)
-		(property "Value" "W25Q128JVE"
+		(property "Value" "AT25SF128A-MHB-T"
 			(at 140.97 109.2199 0)
 			(effects
@@
 			)
 		)
-		(property "Footprint" "Package_SON:WSON-8-1EP_8x6mm_P1.27mm_EP3.4x4.3mm"
+		(property "Footprint" "Package_DFN_QFN:DFN-8-1EP_6x5mm_P1.27mm_EP4x4mm"
 			(at 129.54 85.09 0)
 			(effects
@@
 			)
 		)
-		(property "Datasheet" "https://www.winbond.com/resource-files/w25q128jv_dtr%20revc%2003272018%20plus.pdf"
+		(property "Datasheet" "https://www.renesas.com/en/document/dst/at25sf128aat25qf128a-datasheet?r=1608781"
 			(at 129.54 82.55 0)
 			(effects
@@
 			(at 129.54 107.95 0)
 			(effects
+				(font
+					(size 1.27 1.27)
+				)
+			)
+		)
+		(property "Field4" ""
+			(at 129.54 107.95 0)
+			(effects
