File: Flybot_FC/Flybot FC/src/Flybot_FC/Battery_Monitoring.kicad_sch (KiCad schematic)
At the start: 17 parts, among them J5 Conn_01x02, Q1 IRLML5203TRPBF, Q2 IRLML0100TRPBF, U8 INA219AIDCNR

Commit message: Bill of materials
Parts:
- removed Q1: IRLML5203TRPBF, Package_TO_SOT_SMD:SOT-23, symbol Device:Q_PMOS_GSD
- removed Q2: IRLML0100TRPBF, Package_TO_SOT_SMD:SOT-23, symbol Device:Q_NMOS_GSD
- added Q1: CMLDM7484 TR PBFREE, Package_TO_SOT_SMD:SOT-563, symbol Transistor_FET:FDS4559
- C71: footprint Capacitor_SMD:C_0201_0603Metric -> Capacitor_SMD:C_0402_1005Metric
- D7: footprint LED_SMD:LED_0201_0603Metric -> LED_SMD:LED_0402_1005Metric
- J5: footprint (none) -> greencharge-footprints:CONN_SM02B-SFHLS-TF; symbol Connector_Generic:Conn_01x02 -> Connector_Generic_MountingPin:Conn_01x02_MountingPin
- R25, R26, R32: footprint Resistor_SMD:R_0201_0603Metric -> Resistor_SMD:R_0402_1005Metric
- TP13: footprint (none) -> TestPoint:TestPoint_Pad_D1.0mm
Connections:
- net Batt+: now also Q1.3 (D)
- net GND: now also J5.MP (MountPin), Q1.1 (S)
- net at R24.2, R27.1: now also Q1.5 (G)
- net at R30.1: now also Q1.4 (S)
- net at R27.2: now also Q1.6 (D)
- net at R28.1, R31.1: now also Q1.2 (G)
