File: Flybot_FC/Flybot FC/src/Flybot_FC/ExposedPeripherals.kicad_sch (KiCad schematic)
At the start: 6 parts, among them J4 Conn_02x14_Counter_Clockwise

Commit message: Bill of materials
Parts:
- removed D4: ESDS302DBVR, Package_TO_SOT_SMD:SOT-23-5, symbol Power_Protection:ESDA5V3SC5
- removed J4: Conn_02x14_Counter_Clockwise, symbol Connector_Generic:Conn_02x14_Counter_Clockwise
- added D12, D4: D1213A-01LP4-7B, Diode_SMD:D_0402_1005Metric, symbol Diode:SMAJ78A
- added J4: 1377301, greencharge-footprints:PHOENIX_1377301, symbol Connector_Generic:Conn_02x16_Row_Letter_First
- R22, R23: footprint (none) -> Resistor_SMD:R_0402_1005Metric
Connections:
- net +3V3: now also J4.b1 (Pin_b1), J4.b2 (Pin_b2), J4.b3 (Pin_b3), J4.b4 (Pin_b4), J4.b5 (Pin_b5), J4.b6 (Pin_b6)
- net +5V: now also J4.b7 (Pin_b7), J4.b8 (Pin_b8)
- net CAN1.RX: now also J4.a3 (Pin_a3)
- net CAN1.TX: now also J4.a4 (Pin_a4)
- net ELRS.USART2.RX: now also J4.a5 (Pin_a5)
- net ELRS.USART2.TX: now also J4.a6 (Pin_a6)
- net ESC1: now also J4.b9 (Pin_b9)
- net ESC2: now also J4.b10 (Pin_b10)
- net ESC3: now also J4.b11 (Pin_b11)
- net ESC4: now also J4.b12 (Pin_b12)
- net ESC5: now also J4.b13 (Pin_b13)
- net ESC6: now also J4.b14 (Pin_b14)
- net ESC7: now also J4.b15 (Pin_b15)
- net ESC8: now also J4.b16 (Pin_b16)
- net GND: now also D12.2 (A2), D4.2 (A2), J4.MP, J4.a11 (Pin_a11), J4.a12 (Pin_a12), J4.a13 (Pin_a13), J4.a14 (Pin_a14), J4.a15 (Pin_a15), J4.a16 (Pin_a16)
- net GPS.UART5.RX: now also J4.a7 (Pin_a7)
- net GPS.UART5.TX: now also J4.a8 (Pin_a8)
- net SCL: now also R23.2, D12.1 (A1), J4.a2 (Pin_a2); no longer R22.2
- net SDA: now also R22.2, D4.1 (A1), J4.a1 (Pin_a1); no longer R23.2
- net SPARE.UART8.RX: now also J4.a9 (Pin_a9)
- net SPARE.UART8.TX: now also J4.a10 (Pin_a10)
- no-connect marks 2 -> 0

Commit message: Final Flybot_FC
Connections:
- net +3V3: now also J4.b13 (Pin_b13), J4.b14 (Pin_b14), J4.b15 (Pin_b15), J4.b16 (Pin_b16); no longer J4.b3 (Pin_b3), J4.b4 (Pin_b4), J4.b5 (Pin_b5), J4.b6 (Pin_b6)
- net ESC1: now also J4.b12 (Pin_b12); no longer J4.b9 (Pin_b9)
- net ESC2: now also J4.b11 (Pin_b11); no longer J4.b10 (Pin_b10)
- net ESC3: now also J4.b10 (Pin_b10); no longer J4.b11 (Pin_b11)
- net ESC4: now also J4.b9 (Pin_b9); no longer J4.b12 (Pin_b12)
- net ESC5: now also J4.b3 (Pin_b3); no longer J4.b13 (Pin_b13)
- net ESC6: now also J4.b4 (Pin_b4); no longer J4.b14 (Pin_b14)
- net ESC7: now also J4.b5 (Pin_b5); no longer J4.b15 (Pin_b15)
- net ESC8: now also J4.b6 (Pin_b6); no longer J4.b16 (Pin_b16)
- net SPARE.UART8.RX: now also J4.a10 (Pin_a10); no longer J4.a9 (Pin_a9)
- net SPARE.UART8.TX: now also J4.a9 (Pin_a9); no longer J4.a10 (Pin_a10)
