File: Flybot_FC/Flybot FC/src/Flybot_FC/Flybot_FC.kicad_pcb (KiCad board)
At the start: 2 copper layers, 36 x 36 mm, 196 parts, among them J1 USB_C_Receptacle_USB2.0_16P, J2 SWD interface, J3 Camera, J4 1377301, J5 Conn_01x02, Q1 CMLDM7484 TR PBFREE, Q3 AO3401A, Q4 SI2301CDS-T1-GE3, SW1 SW_Push, U1 STM32F722VCTx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

Commit message: Final Flybot_FC
Parts:
- added G***: LOGO, greencharge-footprints:FlybotLogo, B.Cu at (144.2, 98.5)
- TP22, TP23: moved to B.Cu
- moved TP1 15.9 mm to (144.8, 82.4)
- moved TP3 12.8 mm to (138.9, 82.2)
- moved TP18 11.2 mm to (121.1, 95.4)
- moved TP2 11.0 mm to (142.7, 82.5)
- moved TP17 10.2 mm to (151.3, 106.6)
- moved TP26 7.11 mm to (134.3, 111.4)
- moved R35 6.92 mm to (141.2, 103.0), turned to 0 degrees
- moved R36 3.99 mm to (139.2, 103.0), turned to 180 degrees
- moved TP23 1.80 mm to (132.8, 82.0)
- moved TP20 1.22 mm to (130.8, 80.6)
- moved TP11 1.13 mm to (137.7, 88.4)
- moved Q4 1.08 mm to (138.9, 105.5), turned to 180 degrees
- moved R4 0.83 mm to (144.7, 95.2), turned to 90 degrees
- moved TP22 0.79 mm to (134.3, 81.8)
- moved TP5 0.78 mm to (151.6, 90.1)
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Connections:
- J4 pad a10: /ExposedPeripherals/SPARE.UART8.TX -> /ExposedPeripherals/SPARE.UART8.RX
- J4 pad a9: /ExposedPeripherals/SPARE.UART8.RX -> /ExposedPeripherals/SPARE.UART8.TX
- J4 pad b10: /ExposedPeripherals/ESC2 -> /ExposedPeripherals/ESC3
- J4 pad b11: /ExposedPeripherals/ESC3 -> /ExposedPeripherals/ESC2
- J4 pad b12: /ExposedPeripherals/ESC4 -> /ExposedPeripherals/ESC1
- J4 pad b13: /ExposedPeripherals/ESC5 -> +3V3
- J4 pad b14: /ExposedPeripherals/ESC6 -> +3V3
- J4 pad b15: /ExposedPeripherals/ESC7 -> +3V3
- J4 pad b16: /ExposedPeripherals/ESC8 -> +3V3
- J4 pad b3: +3V3 -> /ExposedPeripherals/ESC5
- J4 pad b4: +3V3 -> /ExposedPeripherals/ESC6
- J4 pad b5: +3V3 -> /ExposedPeripherals/ESC7
- J4 pad b6: +3V3 -> /ExposedPeripherals/ESC8
- J4 pad b9: /ExposedPeripherals/ESC1 -> /ExposedPeripherals/ESC4
- U1 pad 18: /LPS22HBTR_PressureSensor/MEMS2_INT -> unconnected-(U1-PC3-Pad18)
- U1 pad 32: /LSM6DSOX_IMU/IMU1_INT -> unconnected-(U1-PC4-Pad32)
- U1 pad 33: /LSM6DSOX_IMU/IMU2_INT -> unconnected-(U1-PC5-Pad33)
- U1 pad 35: /ML5805_VTX/VTX.XCEN -> unconnected-(U1-PB1-Pad35)
- U1 pad 38: unconnected-(U1-PE8-Pad38) -> /LSM6DSOX_IMU/IMU2_INT
- U1 pad 45: unconnected-(U1-PE15-Pad45) -> /LPS22HBTR_PressureSensor/MEMS2_INT
- U1 pad 51: /LSM6DSOX_IMU/IMU1.CS -> /LSM6DSOX_IMU/IMU2.CS
- U1 pad 53: /STM32F722VC_MCU/Blue LED -> unconnected-(U1-PB14-Pad53)
- U1 pad 60: unconnected-(U1-PD13-Pad60) -> /MAX7456_OSD/LOS
- U1 pad 61: unconnected-(U1-PD14-Pad61) -> /MAX7456_OSD/~{HSYNC}
- U1 pad 62: unconnected-(U1-PD15-Pad62) -> /MAX7456_OSD/~{VSYNC}
- U1 pad 79: /LSM6DSOX_IMU/IMU2.CS -> /STM32F722VC_MCU/Blue LED
- U1 pad 89: /MAX7456_OSD/~{HSYNC} -> unconnected-(U1-PB3-Pad89)
- U1 pad 90: /MAX7456_OSD/~{VSYNC} -> unconnected-(U1-PB4-Pad90)
- U1 pad 91: /MAX7456_OSD/LOS -> /ML5805_VTX/VTX.XCEN
- U1 pad 95: unconnected-(U1-PB8-Pad95) -> /LSM6DSOX_IMU/IMU1_INT
- U1 pad 96: unconnected-(U1-PB9-Pad96) -> /LSM6DSOX_IMU/IMU1.CS
- U3 pad 41: (no net) -> GND
Routing:
- net +3V3: track 0.00 -> 238.4 mm, vias 0 -> 18
- net GND: track 0.00 -> 148.4 mm, vias 0 -> 109
- net +5V: track 0.00 -> 93.0 mm, vias 0 -> 5
- net /SCLK: track 0.00 -> 74.1 mm, vias 0 -> 6
- net /MISO: track 0.00 -> 58.1 mm, vias 0 -> 4
- net /MOSI: track 0.00 -> 54.8 mm, vias 0 -> 6
- net /ExposedPeripherals/SCL: track 0.00 -> 52.2 mm, vias 0 -> 3
- net /ExposedPeripherals/SDA: track 0.00 -> 45.4 mm, vias 0 -> 2
- net /ExposedPeripherals/CAN1.TX: track 0.00 -> 42.5 mm, vias 0 -> 4
- net /MAX7456_OSD/OSD.~{CS}: track 0.00 -> 42.3 mm, vias 0 -> 2
- net /ExposedPeripherals/CAN1.RX: track 0.00 -> 41.1 mm, vias 0 -> 4
- net /MAX7456_OSD/0SD.SCLK: track 0.00 -> 34.1 mm, vias 0 -> 2
- net /MAX7456_OSD/OSD.MOSI: track 0.00 -> 34.1 mm, vias 0 -> 2
- net /STM32F722VC_MCU/NRST: track 0.00 -> 33.5 mm, vias 0 -> 2
- net /ExposedPeripherals/GPS.UART5.TX: track 0.00 -> 31.7 mm, vias 0 -> 3
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- added copper zone on B.Cu, net +3V3
- added copper zone on B.Cu, net +5V
- added copper zone on In1.Cu, net GND
- added copper zone on In2.Cu, net GND
- added copper zone on B.Cu, net Net-(D8-A)
- added copper zone on B.Cu, net Net-(U10-LX)
- added copper zone on B.Cu, net Net-(U9-LX)
Other:
- outline, holes or cut-outs redrawn
- copper layers 2 -> 4
- board text added: "3.3V"
- board text added: "3.3v"
- board text added: "5v"
- board text added: "batt+"
- board text added: "clk"
- board text added: "dio"
- board text added: "gnd"
- board text added: "reset"
- board text added: "rst"
