File: Flybot_FC/Flybot FC/src/Flybot_FC/ML5805_VTX.kicad_sch (KiCad schematic)
At the start: 52 parts, among them U3 ML5805DM, X1 LFB215G37SG8A180

Commit message: Bill of materials
Parts:
- removed C30: 100n, symbol Device:C_Small
- added C86: 100n, Capacitor_SMD:C_0402_1005Metric, symbol Device:C_Small
- AE1: footprint (none) -> Connector_Coaxial:U.FL_Hirose_U.FL-R-SMT-1_Vertical
- C27, C28, C29, C31, C32, C33, C34, C35, C36, C37, C38, C39, C40, C41, C42, C43, C44, C45, C46, C47, C48, C49, C50, C51, C52, C53, C54, C55, C56, C57, C58: footprint (none) -> Capacitor_SMD:C_0402_1005Metric
- L2, L3: footprint (none) -> Inductor_SMD:L_0402_1005Metric
- R14, R15, R16, R17, R18, R19, R21: footprint (none) -> Resistor_SMD:R_0402_1005Metric
- R20: value 400R -> 402R; footprint (none) -> Resistor_SMD:R_0402_1005Metric
- TP10, TP11, TP12, TP6, TP7, TP8, TP9: footprint (none) -> TestPoint:TestPoint_Pad_D1.0mm
- U3: footprint (none) -> Package_DFN_QFN:QFN-40-1EP_6x6mm_P0.5mm_EP4.6x4.6mm
- X1: footprint (none) -> greencharge-footprints:BPF2012LL01R5000A
Connections:
- net +3V3: now also C86.1
- net GND: now also C86.2

Commit message: Final Flybot_FC
Connections:
- net GND renamed EPAD
- net EPAD: now also U3.41 (EPAD)
Changed lines of the file:
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@@
 		(pin "23"
+		)
+		(pin "41"
 		)
 		(instances
