File: Flybot_FC/Flybot FC/src/Flybot_FC/STM32F722VC_MCU.kicad_sch (KiCad schematic)
At the start: 44 parts, among them J1 USB_C_Receptacle_USB2.0_14P, J2 SWD interface, SW1 SW_Push, U1 STM32F722VCTx, Y1 32.768KHz, Y2 8MHz

Commit message: Bill of materials
Parts:
- removed C16, C17: 10p, Capacitor_SMD:C_0201_0603Metric, symbol Device:C_Small
- removed D1: ESDA5V3L, Package_TO_SOT_SMD:SOT-23-3, symbol Power_Protection:ESDA5V3L
- removed J1: USB_C_Receptacle_USB2.0_14P, symbol Connector:USB_C_Receptacle_USB2.0_14P
- removed R5: 2k, Resistor_SMD:R_0201_0603Metric, symbol Device:R_Small_US
- removed Y2: 8MHz, Crystal:Crystal_SMD_3225-4Pin_3.2x2.5mm, symbol Device:Crystal_GND24
- added D1, D11: D1213A-01LP4-7B, Diode_SMD:D_0402_1005Metric, symbol Diode:SMAJ78A
- added J1: USB_C_Receptacle_USB2.0_16P, greencharge-footprints:GCT_USB4216-03-A_REVA, symbol Connector:USB_C_Receptacle_USB2.0_16P
- C1, C10, C11, C12, C13, C18, C19, C2, C3, C4, C5, C6, C7, C8, C9: footprint (none) -> Capacitor_SMD:C_0402_1005Metric
- C14, C15: value 6p -> 12p; footprint Capacitor_SMD:C_0201_0603Metric -> Capacitor_SMD:C_0402_1005Metric
- D2, D3: footprint LED_SMD:LED_0201_0603Metric -> LED_SMD:LED_0402_1005Metric
- J2: footprint (none) -> Connector_PinHeader_2.00mm:PinHeader_1x05_P2.00mm_Vertical
- L1: footprint (none) -> Inductor_SMD:L_0402_1005Metric
- R1, R2, R3, R4: footprint (none) -> Resistor_SMD:R_0402_1005Metric
- R6, R7: footprint Resistor_SMD:R_0201_0603Metric -> Resistor_SMD:R_0402_1005Metric
- SW1: footprint (none) -> greencharge-footprints:SW_SKRPACE010
- TP1, TP2, TP20, TP21, TP22, TP23, TP24, TP3: footprint (none) -> TestPoint:TestPoint_Pad_D1.0mm
Connections:
- net GND: now also D1.2 (A2), D11.2 (A2), J1.A1 (GND), J1.B1 (GND), J1.S1 (SHIELD)
- net USB+: now also D11.1 (A1), J1.A6 (D+), J1.B6 (D+)
- net USB-: now also D1.1 (A1), J1.A7 (D-), J1.B7 (D-)
- net at C10.1, L1.2: now also J1.A4 (VBUS), J1.B4 (VBUS)
- net at R4.1: now also J1.B5 (CC2)
- net at R3.1: now also J1.A5 (CC1)
- net OSC_IN: no longer names the net of U1.12 (PH0)
- net OSC_OUT: no longer names the net of U1.13 (PH1)
- no-connect marks 18 -> 22
Other:
- note removed: "High-speed external clock"

Commit message: Final Flybot_FC
Connections:
- net Blue LED: now also U1.79 (PC11); no longer U1.53 (PB14)
- net IMU1.CS: now also U1.96 (PB9); no longer U1.51 (PB12)
- net IMU1_INT: now also U1.95 (PB8); no longer U1.32 (PC4)
- net IMU2.CS: now also U1.51 (PB12); no longer U1.79 (PC11)
- net IMU2_INT: now also U1.38 (PE8); no longer U1.33 (PC5)
- net LOS: now also U1.60 (PD13); no longer U1.91 (PB5)
- net MEMS2_INT: now also U1.45 (PE15); no longer U1.18 (PC3)
- net VTX.XCEN: now also U1.91 (PB5); no longer U1.35 (PB1)
- net ~{HSYNC}: now also U1.61 (PD14); no longer U1.89 (PB3)
- net ~{VSYNC}: now also U1.62 (PD15); no longer U1.90 (PB4)
